File: 2. Hardware/1. adapter/adapter.kicad_sch (KiCad schematic)
At the start: 1 part, among them U1 LCKFP_GD32F470

Commit message: use all in on adapter
Parts:
- added U2: LoRa, symbol ErBW_s:L33_433UD22S
Other:
- note added: "Copyright (c) 2025, ErBW_s All rights reserved."
Changed lines of the file:
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@@
 	(generator_version "8.0")
 	(paper "A4")
+	(text "Copyright (c) 2025, ErBW_s\nAll rights reserved."
+		(exclude_from_sim no)
+		(at 185.674 179.832 0)
+		(effects
+			(font
+				(size 4.318 4.318)
+			)
+			(justify left bottom)
+		)
+	)
+	(symbol
+		(lib_id "ErBW_s:L33_433UD22S")
+		(at 187.96 59.69 0)
+		(unit 1)
+		(exclude_from_sim no)
+		(in_bom yes)
+		(on_board yes)
+		(dnp no)
+		(fields_autoplaced yes)
+		(property "Reference" "U2"
+			(at 187.96 45.5125 0)
+			(effects
+				(font
+					(size 1.27 1.27)
+				)
+			)
+		)
+		(property "Value" "LoRa"
+			(at 187.96 47.9368 0)
+			(effects
+				(font
+					(size 1.27 1.27)
+				)
+			)
+		)
+		(property "Footprint" ""
+			(at 184.15 55.88 0)
+			(effects
+				(font
+					(size 1.27 1.27)
+				)
+				(hide yes)
+			)
+		)
+		(property "Datasheet" ""
+			(at 184.15 55.88 0)
+			(effects
+				(font
+					(size 1.27 1.27)
+				)
+				(hide yes)
+			)
+		)
+		(property "Description" ""
+			(at 184.15 55.88 0)
+			(effects
+				(font
+					(size 1.27 1.27)
+				)
+				(hide yes)
+			)
+		)
+		(pin "4"
+		)
+		(pin "9"
+		)
+		(pin "7"
+		)
+		(pin "2"
+		)
+		(pin "5"
+		)
+		(pin "10"
+		)
+		(pin "6"
+		)
+		(pin "1"
+		)
+		(pin "8"
+		)
+		(pin "3"
+		)
+		(instances
+			(project ""
+				(path "/94e495b9-aacd-42f9-8fd4-d71efea805b1"
+					(reference "U2")
+					(unit 1)
+				)
+			)
+		)
+	)
 	(symbol
 		(lib_id "ErBW_s:LCKFB_GD32F470")
-		(at 151.13 101.6 0)
+		(at 74.93 54.61 0)
 		(unit 1)
 		(exclude_from_sim no)
@@
 		(fields_autoplaced yes)
 		(property "Reference" "U1"
-			(at 153.035 70.7855 0)
+			(at 76.835 23.7955 0)
 			(effects
 				(font
@@
 		)
 		(property "Value" "LCKFP_GD32F470"
-			(at 153.035 73.2098 0)
+			(at 76.835 26.2198 0)
 			(effects
 				(font
@@
 		)
 		(property "Footprint" ""
-			(at 151.13 72.39 0)
+			(at 74.93 25.4 0)
 			(effects
 				(font
@@
 		)
 		(property "Datasheet" ""
-			(at 151.13 72.39 0)
+			(at 74.93 25.4 0)
 			(effects
 				(font
@@
 		)
 		(property "Description" ""
-			(at 151.13 72.39 0)
-			(effects
-				(font
-					(size 1.27 1.27)
-				)
-				(hide yes)
-			)
+			(at 74.93 25.4 0)
+			(effects
+				(font
+					(size 1.27 1.27)
+				)
+				(hide yes)
+			)
+		)
+		(pin "10"
+		)
+		(pin "1"
+		)
+		(pin "13"
+		)
+		(pin "16"
+		)
+		(pin "14"
+		)
+		(pin "15"
+		)
+		(pin "12"
+		)
+		(pin "11"
+		)
+		(pin "17"
+		)
+		(pin "18"
+		)
+		(pin "19"
+		)
+		(pin "2"
+		)
+		(pin "20"
+		)
+		(pin "21"
 		)
 		(pin "22"
 		)
-		(pin "17"
+		(pin "23"
+		)
+		(pin "24"
+		)
+		(pin "25"
+		)
+		(pin "26"
+		)
+		(pin "27"
+		)
+		(pin "28"
+		)
+		(pin "29"
+		)
+		(pin "3"
+		)
+		(pin "30"
+		)
+		(pin "31"
+		)
+		(pin "32"
+		)
+		(pin "33"
+		)
+		(pin "34"
 		)
 		(pin "35"
@@
 		(pin "36"
 		)
-		(pin "12"
-		)
-		(pin "11"
-		)
-		(pin "25"
-		)
-		(pin "10"
-		)
-		(pin "3"
-		)
-		(pin "30"
+		(pin "37"
+		)
+		(pin "38"
+		)
+		(pin "39"
+		)
+		(pin "69"
+		)
+		(pin "4"
+		)
+		(pin "40"
+		)
+		(pin "41"
+		)
+		(pin "42"
+		)
+		(pin "43"
+		)
+		(pin "44"
+		)
+		(pin "45"
+		)
+		(pin "46"
+		)
+		(pin "47"
+		)
+		(pin "48"
+		)
+		(pin "49"
+		)
+		(pin "5"
+		)
+		(pin "50"
+		)
+		(pin "51"
+		)
+		(pin "52"
+		)
+		(pin "53"
+		)
+		(pin "54"
+		)
+		(pin "55"
+		)
+		(pin "56"
+		)
+		(pin "57"
+		)
+		(pin "58"
+		)
+		(pin "59"
+		)
+		(pin "6"
+		)
+		(pin "60"
+		)
+		(pin "61"
 		)
 		(pin "62"
@@
 		(pin "64"
 		)
-		(pin "15"
-		)
-		(pin "53"
-		)
-		(pin "54"
-		)
-		(pin "55"
-		)
-		(pin "56"
-		)
-		(pin "37"
-		)
-		(pin "38"
-		)
-		(pin "40"
-		)
-		(pin "41"
-		)
-		(pin "69"
+		(pin "65"
+		)
+		(pin "66"
+		)
+		(pin "67"
+		)
+		(pin "68"
 		)
 		(pin "7"
 		)
-		(pin "31"
-		)
-		(pin "32"
-		)
-		(pin "48"
-		)
-		(pin "49"
-		)
-		(pin "46"
-		)
-		(pin "47"
-		)
-		(pin "14"
-		)
-		(pin "28"
-		)
-		(pin "29"
-		)
-		(pin "39"
-		)
-		(pin "4"
-		)
-		(pin "6"
-		)
-		(pin "60"
-		)
-		(pin "61"
-		)
-		(pin "44"
-		)
-		(pin "45"
-		)
-		(pin "42"
-		)
-		(pin "43"
-		)
-		(pin "33"
-		)
-		(pin "34"
+		(pin "70"
+		)
+		(pin "71"
+		)
+		(pin "72"
+		)
+		(pin "73"
+		)
+		(pin "74"
+		)
+		(pin "75"
+		)
+		(pin "76"
+		)
+		(pin "77"
+		)
+		(pin "78"
 		)
 		(pin "79"
@@
 		)
 		(pin "9"
-		)
-		(pin "26"
-		)
-		(pin "27"
-		)
-		(pin "1"
-		)
-		(pin "51"
-		)
-		(pin "52"
-		)
-		(pin "23"
-		)
-		(pin "13"
-		)
-		(pin "24"
-		)
-		(pin "5"
-		)
-		(pin "50"
-		)
-		(pin "20"
-		)
-		(pin "74"
-		)
-		(pin "75"
-		)
-		(pin "76"
-		)
-		(pin "77"
-		)
-		(pin "78"
-		)
-		(pin "2"
-		)
-		(pin "18"
-		)
-		(pin "19"
-		)
-		(pin "16"
-		)
-		(pin "65"
-		)
-		(pin "66"
-		)
-		(pin "67"
-		)
-		(pin "68"
-		)
-		(pin "70"
-		)
-		(pin "71"
-		)
-		(pin "72"
-		)
-		(pin "73"
-		)
-		(pin "57"
-		)
-		(pin "58"
-		)
-		(pin "59"
-		)
-		(pin "21"
 		)
 		(instances
 			(project ""
-				(path "/b23fba04-b800-480a-8334-9433113e049c"
+				(path "/94e495b9-aacd-42f9-8fd4-d71efea805b1"
 					(reference "U1")
 					(unit 1)
